File: 2-digit/2-digit.kicad_pcb (KiCad board)
At the start: 2 copper layers, 27 parts, among them P2 CONN_01X08, U1 74HC595, U4 UDN2981, U5 74HC595, U6 UDN2981, U8 FJS23101AH, U9 FJS23101AH

Commit message: Latest 2-digit PCB
Parts:
- moved R20 76.8 mm to (179.3, 116.5)
- moved R19 76.8 mm to (181.9, 116.5)
- moved R21 76.8 mm to (176.8, 116.5)
- moved C3 66.9 mm to (159.5, 102.6), turned to 90 degrees
- moved C4 65.3 mm to (109.5, 104.6)
- moved C5 65.3 mm to (104.4, 87.4)
- moved P2 65.3 mm to (106.7, 109.2)
- moved R10 65.3 mm to (124.0, 69.6)
- moved R11 65.3 mm to (121.4, 119.6)
- moved R12 65.3 mm to (118.9, 119.6)
- moved R13 65.3 mm to (116.3, 119.6)
- moved R14 65.3 mm to (116.3, 69.6)
- moved R15 65.3 mm to (113.8, 69.6)
- moved R16 65.3 mm to (118.9, 69.6)
- moved R17 65.3 mm to (170.2, 69.4)
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Routing:
- net Net-(R19-Pad1): track 3.58 -> 15.9 mm
- net /SEG2E: track 61.4 -> 49.2 mm
- net /SEG2C: track 58.0 -> 46.3 mm
- net Net-(R20-Pad1): track 3.58 -> 15.2 mm
- net /SEG2D: track 59.4 -> 48.3 mm
- net Net-(R21-Pad1): track 3.58 -> 14.4 mm
- net /LATCH: track 87.0 -> 91.0 mm
- net /CLK: track 90.6 -> 94.6 mm
- net /~OE: track 83.8 -> 87.5 mm
- net +5V: track 84.3 -> 82.3 mm
- net /SEG1C: track 79.2 -> 80.1 mm
- net /SEG1E: track 75.0 -> 75.7 mm
- net /SIG1G: track 26.0 -> 25.3 mm
- net Net-(U1-Pad9): track 39.8 -> 40.5 mm
- net /~CLR: track 95.5 -> 94.9 mm
